Commit message: added warehousing launch file

File: my_rb1_description/urdf/my_rb1_robot.xacro (robot description, xacro)
@@ -2,4 +2,7 @@
 <robot name = "my_rb1_robot" xmlns:xacro="http://www.ros.org/wiki/xacro">
     <xacro:property name="halfpi" value="1.57079632679" />
+    <gazebo reference="base_link">
+        <material>Gazebo/Black</material>
+    </gazebo>
     <joint name="base_joint" type="fixed">
         <parent link="base_link"/>

Commit message: added laser and diff control plugins

File: my_rb1_description/urdf/my_rb1_robot.xacro (robot description, xacro)
@@ -5,4 +5,84 @@
         <material>Gazebo/Black</material>
     </gazebo>
+    <gazebo>
+        <plugin filename="libgazebo_ros_diff_drive.so" name="differential_drive_controller">
+            <alwaysOn>true</alwaysOn>
+            <updateRate>20</updateRate>
+            <leftJoint>lwheel_joint</leftJoint>
+            <rightJoint>rwheel_joint</rightJoint>
+            <wheelSeparation>0.2</wheelSeparation>
+            <wheelDiameter>0.025</wheelDiameter>
+            <torque>10</torque>
+            <commandTopic>cmd_vel</commandTopic>
+            <odometryTopic>odom</odometryTopic>
+            <odometryFrame>odom</odometryFrame>
+            <robotBaseFrame>base_link</robotBaseFrame>
+        </plugin>
+    </gazebo>
+    <gazebo reference="front_caster">
+        <material>Gazebo/Grey</material>
+        <mu1>0</mu1>
+        <mu2>0</mu2>
+    </gazebo>
+    <gazebo reference="back_caster">
+        <material>Gazebo/Grey</material>
+        <mu1>0</mu1>
+        <mu2>0</mu2>
+    </gazebo>
+    <gazebo reference="left_wheel">
+        <material>Gazebo/Red</material>
+        <mu1>1</mu1>
+        <mu2>1</mu2>
+    </gazebo>
+    <gazebo reference="right_wheel">
+        <material>Gazebo/Red</material>
+        <mu1>1</mu1>
+        <mu2>1</mu2>
+    </gazebo>
+    <joint name="laser_joint" type="fixed">
+        <parent link="base_link"/>
+        <axis xyz = "0 1 0"/>
+        <child link="front_laser"/>
+        <origin xyz="0.25 0.0 0.075" rpy="${halfpi*2} 0 0" />
+    </joint>
+    <link name="front_laser">
+    </link>
+    <gazebo reference="front_laser">
+        <sensor type="ray" name="head_hokuyo_sensor">
+            <pose>0 0 0 0 0 0</pose>
+            <visualize>true</visualize>
+            <update_rate>20</update_rate>
+            <alwaysOn>true</alwaysOn>
+            <ray>
+                <scan>
+                    <horizontal>
+                        <samples>720</samples>
+                        <resolution>1</resolution>
+                        <min_angle>-${halfpi}</min_angle>
+                        <max_angle>${halfpi}</max_angle>
+                    </horizontal>
+                </scan>
+                <range>
+                    <min>0.10</min>
+                    <max>10.0</max>
+                    <resolution>0.01</resolution>
+                </range>
+                <noise>
+                    <type>gaussian</type>
+                    <mean>0.0</mean>
+                    <stddev>0.01</stddev>
+                </noise>
+            </ray>
+            <plugin name="gazebo_ros_head_hokuyo_controller" filename="libgazebo_ros_laser.so">
+                <topicName>/laser/scan</topicName>
+                <frameName>front_laser</frameName>
+            </plugin>
+        </sensor>
+    </gazebo>
+    <joint name="dummy_joint" type="fixed">
+        <parent link="dummy"/>
+        <child link="base_link"/>
+    </joint>
+    <link name = "dummy"/>
     <joint name="base_joint" type="fixed">
         <parent link="base_link"/>
@@ -116,5 +196,5 @@
         </visual>
     </link>
-<joint name="bcaster_joint" type="fixed">
+    <joint name="bcaster_joint" type="fixed">
         <parent link="base_link"/>
         <child link="back_caster"/>
@@ -142,11 +222,3 @@
         </visual>
     </link>
-    <joint name="laser_joint" type="fixed">
-        <parent link="base_link"/>
-        <child link="front_laser"/>
-        <origin xyz="0.25 0.0 0.075" rpy="${halfpi*2} 0 0" />
-    </joint>
-    <link name="front_laser">
-        <origin xyz="0 0 0" rpy="0 0 0" />
-    </link>
 </robot>

Commit message: fixed parameters for the diff drive and scan topic

File: my_rb1_description/urdf/my_rb1_robot.xacro (robot description, xacro)
@@ -8,9 +8,10 @@
         <plugin filename="libgazebo_ros_diff_drive.so" name="differential_drive_controller">
             <alwaysOn>true</alwaysOn>
-            <updateRate>20</updateRate>
+            <updateRate>200</updateRate>
             <leftJoint>lwheel_joint</leftJoint>
             <rightJoint>rwheel_joint</rightJoint>
-            <wheelSeparation>0.2</wheelSeparation>
-            <wheelDiameter>0.025</wheelDiameter>
+            <wheelSeparation>0.4</wheelSeparation>
+            <wheelAcceleration>0.5</wheelAcceleration>
+            <wheelDiameter>0.05</wheelDiameter>
             <torque>10</torque>
             <commandTopic>cmd_vel</commandTopic>
@@ -75,5 +76,5 @@
             </ray>
             <plugin name="gazebo_ros_head_hokuyo_controller" filename="libgazebo_ros_laser.so">
-                <topicName>/laser/scan</topicName>
+                <topicName>/scan</topicName>
                 <frameName>front_laser</frameName>
             </plugin>
@@ -121,5 +122,5 @@
         <inertial>
             <origin xyz="0 0 0" rpy="0 0 0" />
-            <mass value="25" />
+            <mass value="1" />
             <inertia ixx="1.5417" ixy="0" ixz="0" iyy="3.467" iyz="0" izz="4.742" />
         </inertial>
@@ -151,5 +152,5 @@
         <inertial>
             <origin xyz="0 0 0" rpy="0 0 0" />
-            <mass value="25" />
+            <mass value="1" />
             <inertia ixx="1.5417" ixy="0" ixz="0" iyy="3.467" iyz="0" izz="4.742" />
         </inertial>
@@ -178,5 +179,5 @@
     <link name="front_caster">
         <inertial>
-            <mass value="25" />
+            <mass value="1" />
             <origin xyz="0 0 0" rpy="0 0 0" />
             <inertia ixx="1.5417" ixy="0" ixz="0" iyy="3.467" iyz="0" izz="4.742" />
@@ -204,5 +205,5 @@
     <link name="back_caster">
         <inertial>
-            <mass value="25" />
+            <mass value="1" />
             <origin xyz="0 0 0" rpy="0 0 0" />
             <inertia ixx="1.5417" ixy="0" ixz="0" iyy="3.467" iyz="0" izz="4.742" />

Commit message: fixed moments of inertia for the small wheels and balls

File: my_rb1_description/urdf/my_rb1_robot.xacro (robot description, xacro)
@@ -94,5 +94,5 @@
     <link name="base_link">
         <inertial>
-            <mass value="25"/>
+            <mass value="23"/>
             <inertia ixx="0.578" ixy="0" ixz="0" iyy="0.578" iyz="0" izz="0.78" />
         </inertial>
@@ -122,6 +122,6 @@
         <inertial>
             <origin xyz="0 0 0" rpy="0 0 0" />
-            <mass value="1" />
-            <inertia ixx="1.5417" ixy="0" ixz="0" iyy="3.467" iyz="0" izz="4.742" />
+            <mass value="0.5" />
+            <inertia ixx="0.000115" ixy="0" ixz="0" iyy="0.000156" iyz="0" izz="0.000115" />
         </inertial>
         <collision>
@@ -152,6 +152,6 @@
         <inertial>
             <origin xyz="0 0 0" rpy="0 0 0" />
-            <mass value="1" />
-            <inertia ixx="1.5417" ixy="0" ixz="0" iyy="3.467" iyz="0" izz="4.742" />
+            <mass value="0.5" />
+            <inertia ixx="0.000115" ixy="0" ixz="0" iyy="0.000156" iyz="0" izz="0.000115" />
         </inertial>
         <collision>
@@ -179,7 +179,7 @@
     <link name="front_caster">
         <inertial>
-            <mass value="1" />
-            <origin xyz="0 0 0" rpy="0 0 0" />
-            <inertia ixx="1.5417" ixy="0" ixz="0" iyy="3.467" iyz="0" izz="4.742" />
+            <mass value="0.5" />
+            <origin xyz="0 0 0" rpy="0 0 0" />
+            <inertia ixx="0.000125" ixy="0" ixz="0" iyy="0.000125" iyz="0" izz="0.000125" />
         </inertial>
         <collision>
@@ -205,7 +205,7 @@
     <link name="back_caster">
         <inertial>
-            <mass value="1" />
-            <origin xyz="0 0 0" rpy="0 0 0" />
-            <inertia ixx="1.5417" ixy="0" ixz="0" iyy="3.467" iyz="0" izz="4.742" />
+            <mass value="0.5" />
+            <origin xyz="0 0 0" rpy="0 0 0" />
+            <inertia ixx="0.000125" ixy="0" ixz="0" iyy="0.000125" iyz="0" izz="0.000125" />
         </inertial>
         <collision>
